File: kicad/MAP4.sch (KiCad schematic (older format))
At the start: 10 parts, among them P1 Logo_MA, P2 Pin

Commit message: MAP4 complete. Boards ordered out
Parts:
- added P3, P4, P5, P6: Pin, map4_fp:MTG_0mm8, symbol CONN_01X01
- D1: value LED Red -> Red
- D2: value LED Grn -> Grn
- D3: value LED Blu -> Blu
- LOGO1: footprint (none) -> map4_fp:Logo_silk_OSHW_6x6mm
- P1: footprint map4_fp:MA_LOGO -> map4_fp:MA_LOGO4
Connections:
- no-connect marks 2 -> 6
Changed lines of the file:
@@
 P 6300 3150
 F 0 "D1" V 6200 3225 50  0000 C CNN
-F 1 "LED Red" H 6300 3050 50  0000 C CNN
+F 1 "Red" H 6300 3050 50  0000 C CNN
 F 2 "map4_fp:LED-5MM" H 6300 3150 50  0001 C CNN
 F 3 "" H 6300 3150 50  0000 C CNN
@@
 P 6800 3175
 F 0 "D2" V 6700 3225 50  0000 C CNN
-F 1 "LED Grn" H 6800 3075 50  0000 C CNN
+F 1 "Grn" H 6800 3075 50  0000 C CNN
 F 2 "map4_fp:LED-5MM" H 6800 3175 50  0001 C CNN
 F 3 "" H 6800 3175 50  0000 C CNN
@@
 P 7300 3175
 F 0 "D3" V 7200 3225 50  0000 C CNN
-F 1 "LED Blu" H 7300 3075 50  0000 C CNN
+F 1 "Blu" H 7300 3075 50  0000 C CNN
 F 2 "map4_fp:LED-5MM" H 7300 3175 50  0001 C CNN
 F 3 "" H 7300 3175 50  0000 C CNN
@@
 F 0 "LOGO1" H 10775 7150 50  0000 C CNN
 F 1 "OPEN_HARDWARE_1" H 10775 6650 50  0000 C CNN
-F 2 "" H 10775 6875 60  0001 C CNN
+F 2 "map4_fp:Logo_silk_OSHW_6x6mm" H 10775 6875 60  0001 C CNN
 F 3 "" H 10775 6875 60  0000 C CNN
 	1    10775 6875
@@
 F 0 "P1" H 7200 6150 50  0000 C CNN
 F 1 "Logo_MA" V 7300 6050 50  0000 C CNN
-F 2 "map4_fp:MA_LOGO" H 7200 6050 50  0001 C CNN
+F 2 "map4_fp:MA_LOGO4" H 7200 6050 50  0001 C CNN
 F 3 "" H 7200 6050 50  0000 C CNN
 	1    7200 6050
@@
 Text Label 7300 3750 1    40   ~ 0
 LED_blu
+$Comp
+L CONN_01X01 P3
+U 1 1 574578C5
+P 8050 6050
+F 0 "P3" H 8050 6150 50  0000 C CNN
+F 1 "Pin" V 8150 6050 50  0000 C CNN
+F 2 "map4_fp:MTG_0mm8" H 8050 6050 50  0001 C CNN
+F 3 "" H 8050 6050 50  0000 C CNN
+	1    8050 6050
+	0    1    1    0
+$EndComp
+NoConn ~ 8050 5850
+$Comp
+L CONN_01X01 P4
+U 1 1 574578FE
+P 8350 6050
+F 0 "P4" H 8350 6150 50  0000 C CNN
+F 1 "Pin" V 8450 6050 50  0000 C CNN
+F 2 "map4_fp:MTG_0mm8" H 8350 6050 50  0001 C CNN
+F 3 "" H 8350 6050 50  0000 C CNN
+	1    8350 6050
+	0    1    1    0
+$EndComp
+NoConn ~ 8350 5850
+$Comp
+L CONN_01X01 P5
+U 1 1 57457995
+P 8650 6050
+F 0 "P5" H 8650 6150 50  0000 C CNN
+F 1 "Pin" V 8750 6050 50  0000 C CNN
+F 2 "map4_fp:MTG_0mm8" H 8650 6050 50  0001 C CNN
+F 3 "" H 8650 6050 50  0000 C CNN
+	1    8650 6050
+	0    1    1    0
+$EndComp
+NoConn ~ 8650 5850
+$Comp
+L CONN_01X01 P6
+U 1 1 5745799C
+P 8950 6050
+F 0 "P6" H 8950 6150 50  0000 C CNN
+F 1 "Pin" V 9050 6050 50  0000 C CNN
+F 2 "map4_fp:MTG_0mm8" H 8950 6050 50  0001 C CNN
+F 3 "" H 8950 6050 50  0000 C CNN
+	1    8950 6050
+	0    1    1    0
+$EndComp
+NoConn ~ 8950 5850
 $EndSCHEMATC

Commit message: Battery holder footprint correction. New Legend
Parts:
- BT1: footprint map4_fp:cr2032_01 -> map4_fp:cr2032_02
Changed lines of the file:
@@
 F 0 "BT1" V 4550 3775 40  0000 L CNN
 F 1 "BATT_HOLDER" V 4550 3200 40  0000 L CNN
-F 2 "map4_fp:cr2032_01" H 4650 3625 60  0001 C CNN
+F 2 "map4_fp:cr2032_02" H 4650 3625 60  0001 C CNN
 F 3 "" H 4650 3625 60  0000 C CNN
 F 4 "HOLDER BATTERY COIN 20MM DIA THM" H 4650 3925 60  0001 L CNN "Field4"
