File: kicad/MAP4.kicad_pcb (KiCad board)
At the start: 2 copper layers, 49.8 x 48.9 mm, 14 parts, among them P1 Logo_MA, P2 Pin, P3 Pin, P4 Pin, P5 Pin, P6 Pin

Commit message: added invert_mask folder for Yellow Mask/Black Legend
Other:
- board text added: "BLACK MASK YELLOW LEGEND"
- board text removed: "PLEASE ADD ETOK MARK TO BOTTOM LAYER ONLY IN THE PROVIDED BOX"
- board text removed: "SPACE FOR ETOK MARK"
Changed lines of the file:
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@@
 (kicad_pcb (version 4) (host pcbnew 4.0.6-e0-6349~53~ubuntu16.04.1)
   (general
-    (links 17)
+    (links 0)
     (no_connects 0)
     (area 111.650001 71.26989 206.380001 126.7)
     (thickness 1.6)
-    (drawings 34)
+    (drawings 66)
     (tracks 64)
     (zones 0)
@@
   )
   (layers
-    (0 F.Cu signal)
-    (31 B.Cu signal)
+    (0 F.Cu signal hide)
+    (31 B.Cu signal hide)
     (32 B.Adhes user)
     (33 F.Adhes user)
@@
     (35 F.Paste user)
     (36 B.SilkS user)
-    (37 F.SilkS user)
+    (37 F.SilkS user hide)
     (38 B.Mask user)
     (39 F.Mask user)
@@
     (zone_45_only no)
     (trace_min 0.2)
-    (segment_width 0.2)
+    (segment_width 0.5)
     (edge_width 0.15)
     (via_size 0.6)
@@
     (visible_elements FFFFEF7F)
     (pcbplotparams
-      (layerselection 0x00130_80000001)
-      (usegerberextensions false)
-      (excludeedgelayer false)
+      (layerselection 0x011f0_80000001)
+      (usegerberextensions true)
+      (usegerberattributes true)
+      (excludeedgelayer true)
       (linewidth 0.050800)
-      (plotframeref true)
+      (plotframeref false)
       (viasonmask false)
       (mode 1)
@@
       (plotvalue true)
       (plotinvisibletext false)
-      (padsonsilk true)
-      (subtractmaskfromsilk false)
-      (outputformat 4)
+      (padsonsilk false)
+      (subtractmaskfromsilk true)
+      (outputformat 1)
       (mirror false)
-      (drillshape 2)
+      (drillshape 0)
       (scaleselection 1)
-      (outputdirectory pdf/))
+      (outputdirectory gerber/))
   )
   (net 0 "")
@@
     )
   )
+  (gr_line (start 148 100) (end 151.5 100) (layer B.SilkS) (width 0.5))
+  (gr_line (start 148 100.5) (end 148 100) (layer B.SilkS) (width 0.5))
+  (gr_line (start 152 100.5) (end 148 100.5) (layer B.SilkS) (width 0.5))
+  (gr_line (start 152 99.5) (end 152 100.5) (layer B.SilkS) (width 0.5))
+  (gr_line (start 147.5 99.5) (end 152 99.5) (layer B.SilkS) (width 0.5))
+  (gr_line (start 147.5 101) (end 147.5 99.5) (layer B.SilkS) (width 0.5))
+  (gr_line (start 152.5 101) (end 147.5 101) (layer B.SilkS) (width 0.5))
+  (gr_line (start 152.5 99) (end 152.5 101) (layer B.SilkS) (width 0.5))
+  (gr_line (start 147 99) (end 152.5 99) (layer B.SilkS) (width 0.5))
+  (gr_line (start 147 101.5) (end 147 99) (layer B.SilkS) (width 0.5))
+  (gr_line (start 153 101.5) (end 147 101.5) (layer B.SilkS) (width 0.5))
+  (gr_line (start 153 98.5) (end 153 101.5) (layer B.SilkS) (width 0.5))
+  (gr_line (start 146.5 98.5) (end 153 98.5) (layer B.SilkS) (width 0.5))
+  (gr_line (start 146.5 102) (end 146.5 98.5) (layer B.SilkS) (width 0.5))
+  (gr_line (start 153.5 102) (end 146.5 102) (layer B.SilkS) (width 0.5))
+  (gr_line (start 153.5 98) (end 153.5 102) (layer B.SilkS) (width 0.5))
+  (gr_line (start 146 98) (end 153.5 98) (layer B.SilkS) (width 0.5))
+  (gr_line (start 146 102.5) (end 146 98) (layer B.SilkS) (width 0.5))
+  (gr_line (start 154 102.5) (end 146 102.5) (layer B.SilkS) (width 0.5))
+  (gr_line (start 154 97.5) (end 154 102.5) (layer B.SilkS) (width 0.5))
+  (gr_line (start 145.5 97.5) (end 154 97.5) (layer B.SilkS) (width 0.5))
+  (gr_line (start 145.5 103) (end 145.5 97.5) (layer B.SilkS) (width 0.5))
+  (gr_line (start 154.5 103) (end 145.5 103) (layer B.SilkS) (width 0.5))
+  (gr_line (start 154.5 97) (end 154.5 103) (layer B.SilkS) (width 0.5))
+  (gr_line (start 145 97) (end 154.5 97) (layer B.SilkS) (width 0.5))
+  (gr_line (start 145 103.5) (end 145 97) (layer B.SilkS) (width 0.5))
+  (gr_line (start 155 103.5) (end 145 103.5) (layer B.SilkS) (width 0.5))
+  (gr_line (start 155 96.5) (end 155 103.5) (layer B.SilkS) (width 0.5))
+  (gr_line (start 144.5 96.5) (end 155 96.5) (layer B.SilkS) (width 0.5))
+  (gr_line (start 144.5 104) (end 144.5 96.5) (layer B.SilkS) (width 0.5))
+  (gr_line (start 155.5 104) (end 144.5 104) (layer B.SilkS) (width 0.5))
+  (gr_line (start 155.5 96) (end 155.5 104) (layer B.SilkS) (width 0.5))
+  (gr_line (start 144 96) (end 155.5 96) (layer B.SilkS) (width 0.5))
   (gr_line (start 173.26 100.18) (end 171.99 98.91) (layer Dwgs.User) (width 0.2))
   (gr_line (start 173.26 97.64) (end 173.26 100.18) (layer Dwgs.User) (width 0.2))
@@
   (gr_line (start 206.28 93.83) (end 206.28 103.99) (layer Dwgs.User) (width 0.2))
   (gr_line (start 177.07 93.83) (end 206.28 93.83) (layer Dwgs.User) (width 0.2))
-  (gr_text "PLEASE ADD ETOK MARK\nTO BOTTOM LAYER ONLY\nIN THE PROVIDED BOX" (at 191.04 98.91) (layer Dwgs.User)
+  (gr_text "BLACK MASK\nYELLOW LEGEND" (at 191.04 98.91) (layer Dwgs.User)
     (effects (font (size 1.5 1.5) (thickness 0.3)))
   )
@@
     (effects (font (size 1 1) (thickness 0.2)) (justify mirror))
   )
-  (gr_line (start 144 95.5) (end 156 95.5) (layer B.SilkS) (width 0.2))
-  (gr_line (start 144 104.5) (end 144 95.5) (layer B.SilkS) (width 0.2))
-  (gr_line (start 156 104.5) (end 144 104.5) (layer B.SilkS) (width 0.2))
-  (gr_line (start 156 95.5) (end 156 104.5) (layer B.SilkS) (width 0.2))
-  (gr_text "SPACE FOR\nETOK MARK" (at 150 93) (layer B.SilkS)
-    (effects (font (size 1.25 1.25) (thickness 0.25)) (justify mirror))
-  )
+  (gr_line (start 144 95.5) (end 156 95.5) (layer B.SilkS) (width 0.5))
+  (gr_line (start 144 104.5) (end 144 95.5) (layer B.SilkS) (width 0.5))
+  (gr_line (start 156 104.5) (end 144 104.5) (layer B.SilkS) (width 0.5))
+  (gr_line (start 156 95.5) (end 156 104.5) (layer B.SilkS) (width 0.5))
   (dimension 49 (width 0.3) (layer Dwgs.User)
     (gr_text "49.000 mm" (at 118.15 96 90) (layer Dwgs.User)
@@
     (arrow2b (pts (xy 125 123.999999) (xy 126.126504 123.413578)))
   )
-  (gr_text [+] (at 139 94.5) (layer B.SilkS)
-    (effects (font (size 1 1) (thickness 0.2)) (justify mirror))
-  )
-  (gr_text [-] (at 162.5 97.5) (layer B.SilkS)
-    (effects (font (size 1 1) (thickness 0.2)) (justify mirror))
+  (gr_text [+] (at 138 95) (layer B.SilkS)
+    (effects (font (size 1.25 1.25) (thickness 0.25)) (justify mirror))
+  )
+  (gr_text [-] (at 162 95) (layer B.SilkS)
+    (effects (font (size 1.25 1.25) (thickness 0.25)) (justify mirror))
   )
   (gr_text "I CAN SOLDER !" (at 150 112.5) (layer B.SilkS)
